Commit message: changed tomasz urdf to be correct package name

File: mxen_ws/src/ourbeloved/urdf/wx250s.urdf.xacro (robot description, xacro)
@@ -7,5 +7,5 @@
   <xacro:property name="pi_offset" value="0.00001"/>
   <material name="interbotix_black">
-    <texture filename="package://vm_sim/mesh/interbotix_black.png"/>
+    <texture filename="package://ourbeloved/mesh/interbotix_black.png"/>
   </material>
   <link name="$(arg robot_name)/$(arg base_link_frame)">
@@ -13,5 +13,5 @@
       <origin rpy="0 0 ${pi/2}" xyz="0 0 0"/>
       <geometry>
-        <mesh filename="package://vm_sim/mesh/wx250s_1_base.stl" scale="0.001 0.001 0.001"/>
+        <mesh filename="package://ourbeloved/mesh/wx250s_1_base.stl" scale="0.001 0.001 0.001"/>
       </geometry>
       <material name="interbotix_black"/>
@@ -29,5 +29,5 @@
       <origin rpy="0 0 ${pi/2}" xyz="0 0 -0.003"/>
       <geometry>
-        <mesh filename="package://vm_sim/mesh/wx250s_2_shoulder.stl" scale="0.001 0.001 0.001"/>
+        <mesh filename="package://ourbeloved/mesh/wx250s_2_shoulder.stl" scale="0.001 0.001 0.001"/>
       </geometry>
       <material name="interbotix_black"/>
@@ -45,5 +45,5 @@
       <origin rpy="0 0 ${pi/2}" xyz="0 0 0"/>
       <geometry>
-        <mesh filename="package://vm_sim/mesh/wx250s_3_upper_arm.stl" scale="0.001 0.001 0.001"/>
+        <mesh filename="package://ourbeloved/mesh/wx250s_3_upper_arm.stl" scale="0.001 0.001 0.001"/>
       </geometry>
       <material name="interbotix_black"/>
@@ -61,5 +61,5 @@
       <origin rpy="0 0 0" xyz="0 0 0"/>
       <geometry>
-        <mesh filename="package://vm_sim/mesh/wx250s_4_upper_forearm.stl" scale="0.001 0.001 0.001"/>
+        <mesh filename="package://ourbeloved/mesh/wx250s_4_upper_forearm.stl" scale="0.001 0.001 0.001"/>
       </geometry>
       <material name="interbotix_black"/>
@@ -77,5 +77,5 @@
       <origin rpy="${pi} 0 0" xyz="0 0 0"/>
       <geometry>
-        <mesh filename="package://vm_sim/mesh/wx250s_5_lower_forearm.stl" scale="0.001 0.001 0.001"/>
+        <mesh filename="package://ourbeloved/mesh/wx250s_5_lower_forearm.stl" scale="0.001 0.001 0.001"/>
       </geometry>
       <material name="interbotix_black"/>
@@ -93,5 +93,5 @@
       <origin rpy="0 0 ${pi/2}" xyz="0 0 0"/>
       <geometry>
-        <mesh filename="package://vm_sim/mesh/wx250s_6_wrist.stl" scale="0.001 0.001 0.001"/>
+        <mesh filename="package://ourbeloved/mesh/wx250s_6_wrist.stl" scale="0.001 0.001 0.001"/>
       </geometry>
       <material name="interbotix_black"/>
@@ -109,5 +109,5 @@
       <origin rpy="0 0 ${pi/2}" xyz="-0.02 0 0"/>
       <geometry>
-        <mesh filename="package://vm_sim/mesh/wx250s_7_gripper.stl" scale="0.001 0.001 0.001"/>
+        <mesh filename="package://ourbeloved/mesh/wx250s_7_gripper.stl" scale="0.001 0.001 0.001"/>
       </geometry>
       <material name="interbotix_black"/>
@@ -133,5 +133,5 @@
       <origin rpy="0 0 ${pi/2}" xyz="-0.0685 0 0"/>
       <geometry>
-        <mesh filename="package://vm_sim/mesh/wx250s_8_gripper_prop.stl" scale="0.001 0.001 0.001"/>
+        <mesh filename="package://ourbeloved/mesh/wx250s_8_gripper_prop.stl" scale="0.001 0.001 0.001"/>
       </geometry>
       <material name="interbotix_black"/>
@@ -148,5 +148,5 @@
       <origin rpy="0 0 ${pi/2}" xyz="-0.063 0 0"/>
       <geometry>
-        <mesh filename="package://vm_sim/mesh/wx250s_9_gripper_bar.stl" scale="0.001 0.001 0.001"/>
+        <mesh filename="package://ourbeloved/mesh/wx250s_9_gripper_bar.stl" scale="0.001 0.001 0.001"/>
       </geometry>
       <material name="interbotix_black"/>
@@ -172,5 +172,5 @@
       <origin rpy="${pi} ${pi} 0" xyz="0 0.005 0"/>
       <geometry>
-        <mesh filename="package://vm_sim/mesh/wx250s_10_gripper_finger.stl" scale="0.001 0.001 0.001"/>
+        <mesh filename="package://ourbeloved/mesh/wx250s_10_gripper_finger.stl" scale="0.001 0.001 0.001"/>
       </geometry>
       <material name="interbotix_black"/>
@@ -189,5 +189,5 @@
       <origin rpy="0 ${pi} 0" xyz="0 -0.005 0"/>
       <geometry>
-        <mesh filename="package://vm_sim/mesh/wx250s_10_gripper_finger.stl" scale="0.001 0.001 0.001"/>
+        <mesh filename="package://ourbeloved/mesh/wx250s_10_gripper_finger.stl" scale="0.001 0.001 0.001"/>
       </geometry>
       <material name="interbotix_black"/>
